Commit message: The sonar plugin was added

File: models/rotors_description/urdf/iris_base.xacro (robot description, xacro)
@@ -91,3 +91,22 @@
     </xacro:bag_plugin_macro>
   </xacro:if>
+  <!-- Downward facing camera -->
+  <xacro:if value="$(arg enable_camera)">
+  <xacro:camera_macro
+    namespace="${namespace}"
+    parent_link="base_link"
+    camera_suffix="bottom"
+    frame_rate="30"
+    horizontal_fov = "81"
+    image_width = "640"
+    image_height = "480"
+    image_format="R8G8B8"
+    min_distance = "0.1"
+    max_distance = "40"
+    noise_mean = "0.0"
+    noise_stddev = "0.0"
+    enable_visual = "true">
+      <origin xyz="0.15 0.0 0.0" rpy="0 ${M_PI/2} 0"/>
+  </xacro:camera_macro>
+  </xacro:if>
 </robot>

Commit message: update iris_base

File: models/rotors_description/urdf/iris_base.xacro (robot description, xacro)
@@ -91,22 +91,22 @@
     </xacro:bag_plugin_macro>
   </xacro:if>
-  <!-- Downward facing camera -->
-  <xacro:if value="$(arg enable_camera)">
-  <xacro:camera_macro
-    namespace="${namespace}"
-    parent_link="base_link"
-    camera_suffix="bottom"
-    frame_rate="30"
-    horizontal_fov = "81"
-    image_width = "640"
-    image_height = "480"
-    image_format="R8G8B8"
-    min_distance = "0.1"
-    max_distance = "40"
-    noise_mean = "0.0"
-    noise_stddev = "0.0"
-    enable_visual = "true">
-      <origin xyz="0.15 0.0 0.0" rpy="0 ${M_PI/2} 0"/>
-  </xacro:camera_macro>
-  </xacro:if>
+  <!-- Downward facing camera
+  <xacro:if value="$(arg enable_camera)">-->
+    <xacro:camera_macro
+      namespace="${namespace}"
+      parent_link="base_link"
+      camera_suffix="bottom"
+      frame_rate="30"
+      horizontal_fov = "81"
+      image_width = "640"
+      image_height = "480"
+      image_format="R8G8B8"
+      min_distance = "0.1"
+      max_distance = "40"
+      noise_mean = "0.0"
+      noise_stddev = "0.0"
+      enable_visual = "true">
+	<origin xyz="0.15 0.0 0.0" rpy="0 ${M_PI/2} 0"/>
+    </xacro:camera_macro>
+  <!--</xacro:if>-->
 </robot>
