Commit message: Update models

File: models/rotors_description/urdf/component_snippets.xacro (robot description, xacro)
@@ -38,10 +38,4 @@
       max_distance noise_mean noise_stddev enable_visual *cylinder *origin">
     <link name="${namespace}/camera_${camera_suffix}_link">
-      <collision>
-        <origin xyz="0 0 0" rpy="0 0 0" />
-        <geometry>
-          <xacro:insert_block name="cylinder" />
-        </geometry>
-      </collision>
       <xacro:if value="${enable_visual}">
         <visual>
@@ -59,8 +53,9 @@
       </inertial>
     </link>
-    <joint name="${namespace}/camera_${camera_suffix}_joint" type="fixed">
+    <joint name="${namespace}/camera_${camera_suffix}_joint" type="revolute">
       <xacro:insert_block name="origin" />
       <parent link="${parent_link}" />
       <child link="${namespace}/camera_${camera_suffix}_link" />
+      <limit upper="0" lower="0" effort="0" velocity="0" />
     </joint>
     <gazebo reference="${namespace}/camera_${camera_suffix}_link">

File: models/rotors_description/urdf/iris_base.xacro (robot description, xacro)
@@ -91,6 +91,6 @@
     </xacro:bag_plugin_macro>
   </xacro:if>
-  <!-- Downward facing camera
-  <xacro:if value="$(arg enable_camera)">-->
+  <!-- Downward facing camera -->
+  <xacro:if value="$(arg enable_camera)">
     <xacro:camera_macro
       namespace="${namespace}"
@@ -98,5 +98,5 @@
       camera_suffix="bottom"
       frame_rate="30"
-      horizontal_fov = "81"
+      horizontal_fov = "1.41"
       image_width = "640"
       image_height = "480"
@@ -107,6 +107,7 @@
       noise_stddev = "0.0"
       enable_visual = "true">
-	<origin xyz="0.15 0.0 0.0" rpy="0 ${M_PI/2} 0"/>
+      <cylinder length="0.01" radius="0.003"/>
+      <origin xyz="0.0 0.0 -0.005" rpy="0 1.57 0"/>
     </xacro:camera_macro>
-  <!--</xacro:if>-->
+  </xacro:if>
 </robot>
